File: pcb/split_flap_unit/split_flap_unit.kicad_pcb (KiCad board)
At the start: 4 copper layers, 39 x 35 mm, 14 parts, among them IC1 ULN2003D1013TR, J1 Main Bus MCU side, J2 Hall, J3 Motor, J4 Main Bus END side, U1 74HC165, U2 74HC595

Commit message: added thermal relief on main pcb and corrected an error
Other:
- board text added: "ESP32 SFU V1.1 Designed by Mathieu Ziegler"
Changed lines of the file:
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@@
 	)
 	(gr_text "JLCJLCJLCJLC\n"
-		(at 160.75 115.5 0)
-		(layer "F.SilkS")
+		(at 177 116 -0)
+		(layer "B.SilkS")
 		(effects
 			(font
@@
 				(bold yes)
 			)
-			(justify left bottom)
+			(justify left bottom mirror)
 		)
 	)
+	(gr_text "ESP32 SFU V1.1\nDesigned by\nMathieu Ziegler\n"
+		(at 176.75 95.25 -0)
+		(layer "B.SilkS")
+		(effects
+			(font
+				(size 1.5 1.5)
+				(thickness 0.3)
+				(bold yes)
+			)
+			(justify left mirror)
+		)
+	)

Commit message: Added text on pcb
Parts:
- renumbered J2 to HALL1, J1 to IN1, J3 to MOTOR1, J4 to OUT1
Routing:
- net GND: vias 60 -> 64
- net +5V: vias 2 -> 1
Other:
- board text added: "GIT"
