File: pcb/split_flap_unit/split_flap_unit.kicad_sch (KiCad schematic)
At the start: 15 parts, among them IC1 ULN2003D1013TR, J1 Main Bus MCU side, J2 Hall, J3 Motor, J4 Main Bus END side, U1 74HC165, U2 74HC595, U3 ESP32-C3_SUPERMINI_SMD

Commit message: added thermal relief on main pcb and corrected an error
Parts:
- removed U3: ESP32-C3_SUPERMINI_SMD, ESP32-C3_SUPERMINI_SMD:MODULE_ESP32-C3_SUPERMINI, symbol ESP32-C3_SUPERMINI_SMD:ESP32-C3_SUPERMINI_SMD

Commit message: Added text on pcb
Parts:
- IC1: DESCRIPTION ULN2003D1013TR, Darlington Transistor Array, NPN 0.5A 50V, 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 -> (none)
- renumbered J2 to HALL1, J1 to IN1, J3 to MOTOR1, J4 to OUT1
